Commit message: Add files via upload

File: bot_4wd/urdf/bot_4wd.xacro (robot description, xacro)
@@ -1,7 +1,7 @@
 <?xml version="1.0" ?>
 <robot name="bot_4wd" xmlns:xacro="http://ros.org/wiki/xacro">
-  <!--xacro:include filename="$(find bot_4wd)/urdf/common_properties.xacro"/>
+  <!--xacro:include filename="$(find bot_4wd)/urdf/common_properties.xacro"/-->
   <xacro:include filename="$(find bot_4wd)/urdf/bot_4wd.gazebo"/>
-    <xacro:include filename="$(find bot_4wd)/urdf/macro.xacro" /-->
+    <!--  xacro:include filename="$(find bot_4wd)/urdf/macro.xacro" /-->
   <link name="base_footprint">
   </link>
@@ -14,5 +14,5 @@
   <link name="base_link">
     <visual>
-      <origin xyz="0 0 0.0" rpy="0 0 0"/>
+      <origin xyz="0 0 0.21" rpy="0 0 0"/>
       <geometry>
         <mesh filename="$(find bot_4wd)/urdf/meshes/base_frame.dae" scale="1 1 1"/>
@@ -34,13 +34,14 @@
     </inertial>
   </link>
+<!--knuckle-->
   <joint name="forward_left_knuckle_joint" type="fixed">
     <parent link="base_link"/>
     <child link="forward_left_knuckle_link"/>
-    <origin xyz="0.0360 -0.036 0.041" rpy="0 0 0"/>
+    <origin xyz="0.4 -0.018 0.12" rpy="0 0 0"/>
     <axis xyz="0 0 1"/>
   </joint>
   <link name="forward_left_knuckle_link">
     <visual>
-      <origin xyz="0 0 0" rpy="0 0 0"/>
+      <origin xyz="0.4 -0.018 0.12" rpy="0 0 0"/>
       <geometry>
         <mesh filename="$(find bot_4wd)/urdf/meshes/knuckle.dae" />
@@ -49,5 +50,5 @@
     </visual>
     <collision>
-      <origin xyz="0 0 0" rpy="0 0 0"/>
+      <origin xyz="0.4 -0.018 0.12" rpy="0 0 0"/>
       <geometry>
       <mesh filename="$(find bot_4wd)/urdf/meshes/knuckle.dae" />
@@ -65,10 +66,10 @@
     <parent link="base_link"/>
     <child link="forward_right_knuckle_link"/>
-    <origin xyz="80.1e-02 -0.036 0.041" rpy="0 0 0"/>
+    <origin xyz="0.4 -0.43 0.12" rpy="0 0 0"/>
     <axis xyz="0 0 1"/>
   </joint>
   <link name="forward_right_knuckle_link">
     <visual>
-      <origin xyz="0 0 0" rpy="0 0 0"/>
+      <origin xyz="0.4 -0.43 0.12" rpy="0 0 0"/>
       <geometry>
         <mesh filename="$(find bot_4wd)/urdf/meshes/knuckle.dae" />
@@ -77,5 +78,5 @@
     </visual>
     <collision>
-      <origin xyz="0 0 0" rpy="0 0 0"/>
+      <origin xyz="0.4 -0.43 0.12" rpy="0 0 0"/>
       <geometry>
       <mesh filename="$(find bot_4wd)/urdf/meshes/knuckle.dae" />
@@ -93,10 +94,10 @@
     <parent link="base_link"/>
     <child link="backward_left_knuckle_link"/>
-    <origin xyz="0.036 -0.8585 0.041" rpy="0 0 0"/>
+    <origin xyz="0.02 -0.018 0.12" rpy="0 0 0"/>
     <axis xyz="0 0 1"/>
   </joint>
   <link name="backward_left_knuckle_link">
     <visual>
-      <origin xyz="0 0 0" rpy="0 0 0"/>
+      <origin xyz="0.02 -0.018 0.12" rpy="0 0 0"/>
       <geometry>
         <mesh filename="$(find bot_4wd)/urdf/meshes/knuckle.dae" />
@@ -105,5 +106,5 @@
     </visual>
     <collision>
-      <origin xyz="0 0 0" rpy="0 0 0"/>
+      <origin xyz="0.02 -0.018 0.12" rpy="0 0 0"/>
       <geometry>
       <mesh filename="$(find bot_4wd)/urdf/meshes/knuckle.dae" />
@@ -121,10 +122,10 @@
     <parent link="base_link"/>
     <child link="backward_right_knuckle_link"/>
-    <origin xyz="80.1e-02 -0.8585 0.041" rpy="0 0 0"/>
+    <origin xyz="0.02 -0.43 0.12" rpy="0 0 0"/>
     <axis xyz="0 0 1"/>
   </joint>
   <link name="backward_right_knuckle_link">
     <visual>
-      <origin xyz="0 0 0" rpy="0 0 0"/>
+      <origin xyz="0.02 -0.43 0.12" rpy="0 0 0"/>
       <geometry>
         <mesh filename="$(find bot_4wd)/urdf/meshes/knuckle.dae" />
@@ -133,5 +134,5 @@
     </visual>
     <collision>
-      <origin xyz="0 0 0" rpy="0 0 0"/>
+      <origin xyz="0.02 -0.43 0.12" rpy="0 0 0"/>
       <geometry>
       <mesh filename="$(find bot_4wd)/urdf/meshes/knuckle.dae" />
@@ -147,41 +148,125 @@
   </link>
 <!-- Wheel-->
-  <joint name="forward_left_wheel_joint" type="fixed">
+  <joint name="forward_left_wheel_joint" type="continuous">
     <parent link="forward_left_knuckle_link"/>
     <child link="forward_left_wheel_link"/>
-    <origin xyz="0.0 -0.0 0.0" rpy="0 0 0"/>
-    <axis xyz="0 0 1"/>
+    <origin xyz="  -0.35 0.05 -0.127" rpy="0 0 0"/>
+    <axis xyz="0 1 0 "/>
   </joint>
   <link name="forward_left_wheel_link">
     <visual>
-      <origin xyz="0 0 0" rpy="0 0 0"/>
-      <geometry>
-        <mesh filename="$(find bot_4wd)/urdf/meshes/wheel.dae" />
-      </geometry>
-      <material name="dark"/>
-    </visual>
-    <collision>
-      <origin xyz="0 0 0" rpy="0 0 0"/>
-      <geometry>
-      <mesh filename="$(find bot_4wd)/urdf/meshes/wheel.dae" />
-      </geometry>
-    </collision>
-    <inertial>
-      <origin xyz="0 0 0" />
-      <mass value="2.8498940e-02" />
-      <inertia ixx="1.1175580e-05" ixy="-4.2369783e-11" ixz="-5.9381719e-09"
-               iyy="1.1192413e-05" iyz="-1.4400107e-11"
-               izz="2.0712558e-05" />
-      </inertial>
-  </link>
-  <joint name="forward_right_wheel_joint" type="fixed">
+      <origin xyz="0 0 0" rpy="1.57 0 0"/>
+      <geometry>
+        <cylinder length="0.1" radius="0.127"/>
+      </geometry>
+      <material name="dark"/>
+    </visual>
+    <collision>
+      <origin xyz="0 0 0" rpy="01.57 0 0"/>
+      <geometry>
+      <cylinder length="0.1" radius="0.127"/>
+      </geometry>
+    </collision>
+    <inertial>
+      <origin xyz="0 0 0" />
+      <mass value="2.8498940e-02" />
+      <inertia ixx="1.1175580e-05" ixy="-4.2369783e-11" ixz="-5.9381719e-09"
+               iyy="1.1192413e-05" iyz="-1.4400107e-11"
+               izz="2.0712558e-05" />
+      </inertial>
+  </link>
+  <joint name="backward_left_wheel_joint" type="continuous">
+    <parent link="backward_left_knuckle_link"/>
+    <child link="backward_left_wheel_link"/>
+    <origin xyz="0.72 0.05 -0.127" rpy="0 0 0"/>
+    <axis xyz="0 1 0 "/>
+  </joint>
+  <link name="backward_left_wheel_link">
+    <visual>
+      <origin xyz="0 0 0" rpy="1.57 0 0"/>
+      <geometry>
+        <cylinder length="0.1" radius="0.127"/>
+      </geometry>
+      <material name="dark"/>
+    </visual>
+    <collision>
+      <origin xyz="0 0 0" rpy="01.57 0 0"/>
+      <geometry>
+      <cylinder length="0.1" radius="0.127"/>
+      </geometry>
+    </collision>
+    <inertial>
+      <origin xyz="0 0 0" />
+      <mass value="2.8498940e-02" />
+      <inertia ixx="1.1175580e-05" ixy="-4.2369783e-11" ixz="-5.9381719e-09"
+               iyy="1.1192413e-05" iyz="-1.4400107e-11"
+               izz="2.0712558e-05" />
+      </inertial>
+  </link>
+  <joint name="forward_right_wheel_joint" type="continuous">
     <parent link="forward_right_knuckle_link"/>
     <child link="forward_right_wheel_link"/>
-    <origin xyz="80.1e-02 -0.0 0.041" rpy="0 0 0"/>
-    <axis xyz="0 0 1"/>
+    <origin xyz="  -0.35 -0.50 -0.127" rpy="0 0 0"/>
+    <axis xyz="0 1 0 "/>
   </joint>
   <link name="forward_right_wheel_link">
     <visual>
-      <origin xyz="0 0 0" rpy="0 0 0"/>
+      <origin xyz="0 0 0" rpy="1.57 0 0"/>
+      <geometry>
+        <cylinder length="0.1" radius="0.127"/>
+      </geometry>
+      <material name="dark"/>
+    </visual>
+    <collision>
+      <origin xyz="0 0 0" rpy="01.57 0 0"/>
+      <geometry>
+      <cylinder length="0.1" radius="0.127"/>
+      </geometry>
+    </collision>
+    <inertial>
+      <origin xyz="0 0 0" />
+      <mass value="2.8498940e-02" />
+      <inertia ixx="1.1175580e-05" ixy="-4.2369783e-11" ixz="-5.9381719e-09"
+               iyy="1.1192413e-05" iyz="-1.4400107e-11"
+               izz="2.0712558e-05" />
+      </inertial>
+  </link>
+  <joint name="backward_right_wheel_joint" type="continuous">
+    <parent link="backward_right_knuckle_link"/>
+    <child link="backward_right_wheel_link"/>
+    <origin xyz="0.72 -0.50 -0.127" rpy="0 0 0"/>
+    <axis xyz="0 1 0 "/>
+  </joint>
+  <link name="backward_right_wheel_link">
+    <visual>
+      <origin xyz="0 0 0" rpy="1.57 0 0"/>
+      <geometry>
+        <cylinder length="0.1" radius="0.127"/>
+      </geometry>
+      <material name="dark"/>
+    </visual>
+    <collision>
+      <origin xyz="0 0 0" rpy="01.57 0 0"/>
+      <geometry>
+      <cylinder length="0.1" radius="0.127"/>
+      </geometry>
+    </collision>
+    <inertial>
+      <origin xyz="0 0 0" />
+      <mass value="2.8498940e-02" />
+      <inertia ixx="1.1175580e-05" ixy="-4.2369783e-11" ixz="-5.9381719e-09"
+               iyy="1.1192413e-05" iyz="-1.4400107e-11"
+               izz="2.0712558e-05" />
+      </inertial>
+  </link>
+  <!--joint name="forward_right_wheel_joint" type="continuous">
+    <parent link="forward_right_knuckle_link"/>
+    <child link="forward_right_wheel_link"/>
+    <origin xyz="0.151 -0.22 -0.13" rpy="0 0 0"/>
+    <axis xyz="0 1 0"/>
+  </joint>
+  <link name="forward_right_wheel_link">
+    <visual>
+      <origin xyz="0.151 -0.22 -0.13" rpy="0 0 0"/>
       <geometry>
         <mesh filename="$(find bot_4wd)/urdf/meshes/wheel.dae" />
@@ -190,5 +275,5 @@
     </visual>
     <collision>
-      <origin xyz="0 0 0" rpy="0 0 0"/>
+      <origin xyz="0.151 -0.22 -0.13" rpy="0 0 0"/>
       <geometry>
       <mesh filename="$(find bot_4wd)/urdf/meshes/wheel.dae" />
@@ -203,13 +288,13 @@
       </inertial>
   </link>
-  <joint name="backward_left_wheel_joint" type="fixed">
+  <joint name="backward_left_wheel_joint" type="continuous">
     <parent link="backward_left_knuckle_link"/>
     <child link="backward_left_wheel_link"/>
-    <origin xyz="0.0 -0.8525 0.041" rpy="0 0 0"/>
-    <axis xyz="0 0 1"/>
+    <origin xyz="-0.05 0.045 -0.13" rpy="0 0 0"/>
+    <axis xyz="0 1 0 "/>
   </joint>
   <link name="backward_left_wheel_link">
     <visual>
-      <origin xyz="0 0 0" rpy="0 0 0"/>
+      <origin xyz="-0.05 0.045 -0.13" rpy="0 0 0"/>
       <geometry>
         <mesh filename="$(find bot_4wd)/urdf/meshes/wheel.dae" />
@@ -218,5 +303,5 @@
     </visual>
     <collision>
-      <origin xyz="0 0 0" rpy="0 0 0"/>
+      <origin xyz="-0.05 0.045 -0.13" rpy="0 0 0"/>
       <geometry>
       <mesh filename="$(find bot_4wd)/urdf/meshes/wheel.dae" />
@@ -231,13 +316,13 @@
       </inertial>
   </link>
-  <joint name="backward_right_wheel_joint" type="fixed">
+  <joint name="backward_right_wheel_joint" type="continuous">
     <parent link="backward_right_knuckle_link"/>
     <child link="backward_right_wheel_link"/>
-    <origin xyz="80.1e-02 -0.8725 0.041" rpy="0 0 0"/>
-    <axis xyz="0 0 1"/>
+    <origin xyz="-0.05 -0.22 -0.13" rpy="0 0 0"/>
+    <axis xyz="0 1 0"/>
   </joint>
   <link name="backward_right_wheel_link">
     <visual>
-      <origin xyz="0 0 0" rpy="0 0 0"/>
+      <origin xyz="-0.05 -0.22 -0.13" rpy="0 0 0"/>
       <geometry>
         <mesh filename="$(find bot_4wd)/urdf/meshes/wheel.dae" />
@@ -246,5 +331,5 @@
     </visual>
     <collision>
-      <origin xyz="0 0 0" rpy="0 0 0"/>
+      <origin xyz="-0.05 -0.22 -0.13" rpy="0 0 0"/>
       <geometry>
       <mesh filename="$(find bot_4wd)/urdf/meshes/wheel.dae" />
@@ -258,4 +343,4 @@
                izz="2.0712558e-05" />
       </inertial>
-  </link>
+  </link-->
 </robot>

File: bot_4wd/urdf/bot_4wd_test.xacro (robot description, xacro)
@@ -34,4 +34,5 @@
     </inertial>
   </link>
+<!--knuckle-->
   <joint name="forward_left_knuckle_joint" type="fixed">
     <parent link="base_link"/>
@@ -147,8 +148,8 @@
   </link>
 <!-- Wheel-->
-  <joint name="forward_left_wheel_joint" type="fixed">
-    <parent link="base_link"/>
+  <joint name="forward_left_wheel_joint" type="continuous">
+    <parent link="forward_left_knuckle_link"/>
     <child link="forward_left_wheel_link"/>
-    <origin xyz="0.0360 -0.050 0.041" rpy="0 0 0"/>
+    <origin xyz="0.0 -0.0 0.0" rpy="0 0 0"/>
     <axis xyz="0 0 1"/>
   </joint>
@@ -175,8 +176,8 @@
       </inertial>
   </link>
-  <joint name="forward_right_wheel_joint" type="fixed">
-    <parent link="base_link"/>
+  <joint name="forward_right_wheel_joint" type="continuous">
+    <parent link="forward_right_knuckle_link"/>
     <child link="forward_right_wheel_link"/>
-    <origin xyz="80.1e-02 -0.050 0.041" rpy="0 0 0"/>
+    <origin xyz="0 0 0" rpy="0 0 0"/>
     <axis xyz="0 0 1"/>
   </joint>
@@ -203,8 +204,8 @@
       </inertial>
   </link>
-  <joint name="backward_left_wheel_joint" type="fixed">
-    <parent link="base_link"/>
+  <joint name="backward_left_wheel_joint" type="continuous">
+    <parent link="backward_left_knuckle_link"/>
     <child link="backward_left_wheel_link"/>
-    <origin xyz="0.036 -0.8525 0.041" rpy="0 0 0"/>
+    <origin xyz="0.0 -0 0" rpy="0 0 0"/>
     <axis xyz="0 0 1"/>
   </joint>
@@ -231,8 +232,8 @@
       </inertial>
   </link>
-  <joint name="backward_right_wheel_joint" type="fixed">
-    <parent link="base_link"/>
+  <joint name="backward_right_wheel_joint" type="continuous">
+    <parent link="backward_right_knuckle_link"/>
     <child link="backward_right_wheel_link"/>
-    <origin xyz="80.1e-02 -0.8725 0.041" rpy="0 0 0"/>
+    <origin xyz="0 0 0" rpy="0 0 0"/>
     <axis xyz="0 0 1"/>
   </joint>
